File: TFT_LCD_Display_EC11_Board.kicad_pcb (KiCad board)
At the start: 2 copper layers, 91 x 44 mm, 39 parts, among them J1 USB_C_Receptacle_USB2.0_16P, J2 Control, J3 I2C, J4 TFT-LCD-DISPLAY-EC11, Q1 BC848, Q2 BC848, SW1 BOOT, SW2 EN, U1 MCP1826S, U2 USBLC6-2SC6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

Commit message: Rev.2.1 and openScad files
Parts:
- added R11: 10k, Resistor_SMD:R_1206_3216Metric_Pad1.30x1.75mm_HandSolder, F.Cu at (158.0, 88.0)
- moved C4 2.09 mm to (158.0, 94.0)
Routing:
- net 3v3: track 199.5 -> 294.8 mm, vias 2 -> 8
- net VBUS: track 100.9 -> 159.0 mm
- net SCL: track 60.2 -> 109.8 mm
- net ESP-RX: track 62.7 -> 107.8 mm
- net GPIO0: track 91.5 -> 130.4 mm
- net ESP-TX: track 63.8 -> 91.7 mm
- net B: track 32.4 -> 53.8 mm
- net SDA: track 51.4 -> 68.5 mm
- net ~{DTR}: track 31.0 -> 47.0 mm
- net K0: track 37.5 -> 53.2 mm
- net A: track 31.3 -> 46.4 mm
- net RESET: track 49.4 -> 63.1 mm, vias 1 -> 3
- net RES: track 29.6 -> 42.8 mm
- net PUSH: track 36.7 -> 49.8 mm
- net Net-(U4-V3): track 10.5 -> 18.3 mm
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Other:
- board text added: "Rev.2.1 [16-05-2026]"
- board text removed: "Rev.2.0 [06-05-2026]"
