File: TFT_LCD_Display_EC11_Board.kicad_sch (KiCad schematic)
At the start: 39 parts, among them J1 USB_C_Receptacle_USB2.0_16P, J2 Control, J3 I2C, J4 TFT-LCD-DISPLAY-EC11, Q1 BC848, Q2 BC848, SW1 BOOT, SW2 EN, U1 MCP1826S, U2 USBLC6-2SC6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

Commit message: Rev.2.1 and openScad files
Parts:
- added R11: 10k, Resistor_SMD:R_1206_3216Metric_Pad1.30x1.75mm_HandSolder, symbol Device:R
Connections:
- net 3v3: now also R11.2
- net ~{ENABLE}: now also R11.1
Other:
- moved on the sheet: R6
Changed lines of the file:
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@@
 	(title_block
 		(title "TFT LCD Display EC11 ESP32 Board")
-		(date "2026-05-06")
-		(rev "r2.0")
+		(date "2026-05-16")
+		(rev "r2.1")
 		(company "by Willem Aandewiel")
+		(comment 1 "r2.1: new R11 (pullup ENABLE pin)")
 	)
 	(rectangle
@@
 	)
 	(rectangle
-		(start 93.98 110.49)
+		(start 87.63 110.49)
 		(end 169.545 187.96)
 		(stroke
@@
 	)
 	(junction
-		(at 110.49 147.32)
-		(diameter 0)
-		(color 0 0 0 0)
-	)
-	(junction
 		(at 72.39 29.21)
 		(diameter 0)
@@
 	)
 	(junction
+		(at 110.49 147.32)
+		(diameter 0)
+		(color 0 0 0 0)
+	)
+	(junction
 		(at 116.84 69.85)
 		(diameter 0)
@@
 	(wire
 		(pts
+			(xy 106.68 125.73) (xy 106.68 127)
+		)
+		(stroke
+			(width 0)
+			(type default)
+		)
+	)
+	(wire
+		(pts
 			(xy 99.06 69.85) (xy 106.68 69.85)
 		)
@@
 	(wire
 		(pts
-			(xy 109.22 151.13) (xy 110.49 151.13)
+			(xy 107.95 151.13) (xy 110.49 151.13)
 		)
 		(stroke
@@
 	(global_label "3v3"
 		(shape input)
-		(at 101.6 151.13 180)
+		(at 100.33 151.13 180)
 		(fields_autoplaced yes)
 		(effects
@@
 		)
 		(property "Intersheetrefs" "${INTERSHEET_REFS}"
-			(at 95.2282 151.13 0)
+			(at 93.9582 151.13 0)
 			(hide yes)
 			(show_name no)
@@
 		)
 	)
+	(global_label "3v3"
+		(shape input)
+		(at 106.68 118.11 90)
+		(fields_autoplaced yes)
+		(effects
+			(font
+				(size 1.27 1.27)
+			)
+			(justify left)
+		)
+		(property "Intersheetrefs" "${INTERSHEET_REFS}"
+			(at 106.68 111.7382 90)
+			(hide yes)
+			(show_name no)
+			(do_not_autoplace no)
+			(effects
+				(font
+					(size 1.27 1.27)
+				)
+				(justify left)
+			)
+		)
+	)
 	(global_label "~{ENABLE}"
 		(shape input)
@@
 	)
 	(symbol
+		(lib_id "Device:R")
+		(at 106.68 121.92 180)
+		(unit 1)
+		(body_style 1)
+		(exclude_from_sim no)
+		(in_bom yes)
+		(on_board yes)
+		(in_pos_files yes)
+		(dnp no)
+		(property "Reference" "R11"
+			(at 104.648 122.428 90)
+			(show_name no)
+			(do_not_autoplace no)
+			(effects
+				(font
+					(size 1.27 1.27)
+				)
+			)
+		)
+		(property "Value" "10k"
+			(at 108.712 121.92 90)
+			(show_name no)
+			(do_not_autoplace no)
+			(effects
+				(font
+					(size 1.27 1.27)
+				)
+			)
+		)
+		(property "Footprint" "Resistor_SMD:R_1206_3216Metric_Pad1.30x1.75mm_HandSolder"
+			(at 108.458 121.92 90)
+			(hide yes)
+			(show_name no)
+			(do_not_autoplace no)
+			(effects
+				(font
+					(size 1.27 1.27)
+				)
+			)
+		)
+		(property "Datasheet" ""
+			(at 106.68 121.92 0)
+			(hide yes)
+			(show_name no)
+			(do_not_autoplace no)
+			(effects
+				(font
+					(size 1.27 1.27)
+				)
+			)
+		)
+		(property "Description" "Resistor"
+			(at 106.68 121.92 0)
+			(hide yes)
+			(show_name no)
+			(do_not_autoplace no)
+			(effects
+				(font
+					(size 1.27 1.27)
+				)
+			)
+		)
+		(pin "1"
+		)
+		(pin "2"
+		)
+		(instances
+			(project "TFT_LCD_Display_EC11_Board"
+				(path "/3c59e70f-e9c5-4ef4-a932-269e9554ea5b"
+					(reference "R11")
+					(unit 1)
+				)
+			)
+		)
+	)
+	(symbol
 		(lib_id "Connector:Conn_01x12_Socket")
 		(at 259.08 142.24 0)
@@
 	(symbol
 		(lib_id "Device:R")
-		(at 105.41 151.13 270)
+		(at 104.14 151.13 270)
 		(unit 1)
 		(body_style 1)
@@
 		(dnp no)
 		(property "Reference" "R6"
-			(at 105.918 153.162 90)
+			(at 104.648 153.162 90)
 			(show_name no)
 			(do_not_autoplace no)
@@
 		)
 		(property "Value" "10k"
-			(at 105.41 149.098 90)
+			(at 104.14 149.098 90)
 			(show_name no)
 			(do_not_autoplace no)
@@
 		)
 		(property "Footprint" "Resistor_SMD:R_1206_3216Metric_Pad1.30x1.75mm_HandSolder"
-			(at 105.41 149.352 90)
+			(at 104.14 149.352 90)
 			(hide yes)
 			(show_name no)
@@
 		)
 		(property "Datasheet" ""
-			(at 105.41 151.13 0)
+			(at 104.14 151.13 0)
 			(hide yes)
 			(show_name no)
@@
 		)
 		(property "Description" "Resistor"
-			(at 105.41 151.13 0)
+			(at 104.14 151.13 0)
 			(hide yes)
 			(show_name no)
